File: pcb/Electra/Electra2-bu.kicad_pcb (KiCad board)
At the start: 2 copper layers, 100 x 48.5 mm, 79 parts, among them J101 RTC, J102 UART, J201 8-28VIn, J202 USB_B_Micro, J203 Enable VIn, J301 Relay2/D, J401 Relay1/U, J501 S1/U, J502 S2/D, J701 A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

Commit message: PCB Ver 1 completed (TODO: Check)
Parts:
- D302, D402: value 200mA -> DIODE
- J301: value Relay2/D -> Relay1/U
- J401: value Relay1/U -> Relay2/D
- J502: value S2/D -> SW2/D
- R201, R202, R204, R205, R206: footprint Resistor_SMD:R_0603_1608Metric_Pad0.98x0.95mm_HandSolder -> Resistor_SMD:R_0201_0603Metric_Pad0.64x0.40mm_HandSolder
- moved C207 3.97 mm to (100.0, 107.3)
- moved R206 3.65 mm to (101.8, 108.3)
- moved R205 3.11 mm to (101.8, 107.3)
- moved R204 2.57 mm to (101.8, 106.3)
- moved R202 2.04 mm to (101.8, 105.3)
- moved R201 1.56 mm to (101.8, 104.3)
Routing:
- net Net-(C207-Pad1): track 10.6 -> 7.01 mm
- net Net-(C201-Pad1): track 2.93 -> 0.09 mm
- net Net-(R201-Pad2): track 7.74 -> 5.86 mm, vias 0 -> 2
- net Net-(C207-Pad2): track 3.33 -> 2.40 mm
- net Net-(J601-Pad4): vias 1 -> 0
