File: pcb/Electra/Electra_bu2.kicad_pcb (KiCad board)
At the start: 2 copper layers, 100 x 48.5 mm, 76 parts, among them J101 Extra1, J102 RTC, J103 Extra2, J104 UART, J201 USB, J202 7-12V, J301 Relay 2/D, J401 S1/U, J402 S2/D, J601 A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

Commit message: Rev 2 completed, todo check all and remove not needed filed
Parts:
- removed the G*** at (176.9, 92.1)
- removed the G*** at (194.0, 103.5)
- added G***: LOGO, Custom:Electricity-Causion-6.1mmX6.1mm-logo, B.Cu at (176.8, 92.0)
- added G***: LOGO, Custom:Electricity-Causion-6.1mmX6.1mm-logo, F.Cu at (193.8, 103.4)
- moved TP202 2.23 mm to (104.1, 93.4)
- moved R701 0.30 mm to (155.5, 82.5)
- moved G*** 0.17 mm to (99.4, 78.9)
- renumbered J202 to Je
Routing:
- net Net-(C201-Pad1): track 6.95 -> 0.07 mm
- net /ESP8266/GPIO0: track 58.3 -> 61.7 mm
- net +3V3: track 177.4 -> 175.6 mm
- net /Extra1: track 70.8 -> 71.9 mm
- net /TX: track 50.8 -> 51.4 mm
- net GND: vias 391 -> 366
- net (no net): vias 6 -> 7
Other:
- outline, holes or cut-outs redrawn
- board text added: "7-12V"
- board text added: "Vin"
- board text removed: "+"
- board text removed: "10"
- board text removed: "2"
- board text removed: "Data"
- board text removed: "If you are reading this, I hope you have a nice day!"
- board text removed: "SDA"
- board text removed: "SDL"
