File: pcb/Electra/ESP8266.sch (KiCad schematic (older format))
At the start: 16 parts, among them J601 Conn_01x06_Female, SW601 SW_MEC_5G, SW602 SW_MEC_5G, U601 ESP-12F

Commit message: PCB Ver 1 completed (TODO: Check)
Parts:
- removed SW601, SW602: SW_MEC_5G, Button_Switch_SMD:SW_SPST_EVQPE1, symbol Switch:SW_MEC_5G
- added SW601, SW602: SW_Push, Button_Switch_SMD:SW_SPST_EVQPE1, symbol Switch:SW_Push
- R604, R607: Description 80.6Ω ±1% 0.1W ±100ppm/℃ 0603 Chip Resistor - Surface Mount RoHS -> 80.6Ω ±1% 0.1W ±100ppm/℃ 0603 Chip Resistor - Surface Mount RoHS
Connections:
- net GPIO0: now also SW601.2
- net ~RST: now also SW602.2
- net GNDREF renamed GND
- net GND: now also SW601.1, SW602.1

Commit message: PCB completed (added silkscreen more)
Parts:
- D601: value LED -> TX; Mfr.Part # NCD0603Y1 -> KT-0603R
- D602: value LED -> RX; Mfr.Part # NCD0603Y1 -> KT-0603R
- J601: value Conn_01x06_Female -> FTDI
- JP601: value Jumper_NC_Small -> Power
- SW601: value SW_Push -> Flash
- SW602: value SW_Push -> RST
Changed lines of the file:
@@
 P 10450 5150
 F 0 "J601" H 10350 4750 50  0000 L CNN
-F 1 "Conn_01x06_Female" V 10650 4950 50  0000 L CNN
+F 1 "FTDI" H 10300 5500 50  0000 L CNN
 F 2 "Connector_PinHeader_2.54mm:PinHeader_1x06_P2.54mm_Vertical" H 10450 5150 50  0001 C CNN
 F 3 "-" H 10450 5150 50  0001 C CNN
@@
 	-1   0    0    1
 $EndComp
-$Comp
-L Device:LED D602
-U 1 1 608DFB8B
-P 8000 5250
-F 0 "D602" V 8050 5150 50  0000 R CNN
-F 1 "LED" V 7950 5150 50  0000 R CNN
-F 2 "LED_SMD:LED_0603_1608Metric_Pad1.05x0.95mm_HandSolder" H 8000 5250 50  0001 C CNN
-F 3 "https://datasheet.lcsc.com/szlcsc/2008201033_Foshan-NationStar-Optoelectronics-NCD0603Y1_C84268.pdf" H 8000 5250 50  0001 C CNN
-F 4 "Yellow 586~595nm 0603 Light Emitting Diodes (LED) RoHS" H 8000 5250 50  0001 C CNN "Description"
-F 5 "C84268" H 8000 5250 50  0001 C CNN "LCSC Part #"
-F 6 "Foshan NationStar Optoelectronics" H 8000 5250 50  0001 C CNN "Manufacturer"
-F 7 "15mA" H 8000 5250 50  0001 C CNN "Maximum Value"
-F 8 "NCD0603Y1" H 8000 5250 50  0001 C CNN "Mfr.Part #"
-F 9 "0603" H 8000 5250 50  0001 C CNN "Package Reference"
-	1    8000 5250
-	0    -1   -1   0
-$EndComp
 Wire Wire Line
 	8000 5950 8000 5400
@@
 Wire Wire Line
 	6150 5950 6150 5450
-$Comp
-L Device:LED D601
-U 1 1 608DE81B
-P 6150 5300
-F 0 "D601" V 6200 5200 50  0000 R CNN
-F 1 "LED" V 6100 5200 50  0000 R CNN
-F 2 "LED_SMD:LED_0603_1608Metric_Pad1.05x0.95mm_HandSolder" H 6150 5300 50  0001 C CNN
-F 3 "https://datasheet.lcsc.com/szlcsc/2008201033_Foshan-NationStar-Optoelectronics-NCD0603Y1_C84268.pdf" H 6150 5300 50  0001 C CNN
-F 4 "Yellow 586~595nm 0603 Light Emitting Diodes (LED) RoHS" H 6150 5300 50  0001 C CNN "Description"
-F 5 "C84268" H 6150 5300 50  0001 C CNN "LCSC Part #"
-F 6 "Foshan NationStar Optoelectronics" H 6150 5300 50  0001 C CNN "Manufacturer"
-F 7 "15mA" H 6150 5300 50  0001 C CNN "Maximum Value"
-F 8 "NCD0603Y1" H 6150 5300 50  0001 C CNN "Mfr.Part #"
-F 9 "0603" H 6150 5300 50  0001 C CNN "Package Reference"
-	1    6150 5300
-	0    -1   -1   0
-$EndComp
 Wire Wire Line
 	6150 5150 6150 5100
@@
 U 1 1 60C67B52
 P 9800 4750
-F 0 "JP601" V 9850 5550 50  0000 R CNN
-F 1 "Jumper_NC_Small" V 9750 5550 50  0000 R CNN
+F 0 "JP601" V 9850 5150 50  0000 R CNN
+F 1 "Power" V 9750 5150 50  0000 R CNN
 F 2 "Jumper:SolderJumper-2_P1.3mm_Bridged_RoundedPad1.0x1.5mm" H 9800 4750 50  0001 C CNN
 F 3 "-" H 9800 4750 50  0001 C CNN
@@
 P 1650 5350
 F 0 "SW601" V 1696 5302 50  0000 R CNN
-F 1 "SW_Push" V 1605 5302 50  0000 R CNN
+F 1 "Flash" V 1605 5302 50  0000 R CNN
 F 2 "Button_Switch_SMD:SW_SPST_EVQPE1" H 1650 5550 50  0001 C CNN
 F 3 "https://datasheet.lcsc.com/szlcsc/2005221232_SHOU-HAN-TS342A2P-WZ_C557591.pdf" H 1650 5550 50  0001 C CNN
@@
 P 4050 5250
 F 0 "SW602" V 4096 5202 50  0000 R CNN
-F 1 "SW_Push" V 4005 5202 50  0000 R CNN
+F 1 "RST" V 4005 5202 50  0000 R CNN
 F 2 "Button_Switch_SMD:SW_SPST_EVQPE1" H 4050 5450 50  0001 C CNN
 F 3 "https://datasheet.lcsc.com/szlcsc/2005221232_SHOU-HAN-TS342A2P-WZ_C557591.pdf" H 4050 5450 50  0001 C CNN
@@
 Wire Wire Line
 	5750 3250 5750 3550
+$Comp
+L Device:LED D601
+U 1 1 608DE81B
+P 6150 5300
+F 0 "D601" V 6200 5200 50  0000 R CNN
+F 1 "TX" V 6100 5200 50  0000 R CNN
+F 2 "LED_SMD:LED_0603_1608Metric_Pad1.05x0.95mm_HandSolder" H 6150 5300 50  0001 C CNN
+F 3 "https://datasheet.lcsc.com/szlcsc/2008201033_Foshan-NationStar-Optoelectronics-NCD0603Y1_C84268.pdf" H 6150 5300 50  0001 C CNN
+F 4 "Yellow 586~595nm 0603 Light Emitting Diodes (LED) RoHS" H 6150 5300 50  0001 C CNN "Description"
+F 5 "C84268" H 6150 5300 50  0001 C CNN "LCSC Part #"
+F 6 "Foshan NationStar Optoelectronics" H 6150 5300 50  0001 C CNN "Manufacturer"
+F 7 "15mA" H 6150 5300 50  0001 C CNN "Maximum Value"
+F 8 "KT-0603R" H 6150 5300 50  0001 C CNN "Mfr.Part #"
+F 9 "0603" H 6150 5300 50  0001 C CNN "Package Reference"
+	1    6150 5300
+	0    -1   -1   0
+$EndComp
+$Comp
+L Device:LED D602
+U 1 1 608DFB8B
+P 8000 5250
+F 0 "D602" V 8050 5150 50  0000 R CNN
+F 1 "RX" V 7950 5150 50  0000 R CNN
+F 2 "LED_SMD:LED_0603_1608Metric_Pad1.05x0.95mm_HandSolder" H 8000 5250 50  0001 C CNN
+F 3 "https://datasheet.lcsc.com/szlcsc/2008201033_Foshan-NationStar-Optoelectronics-NCD0603Y1_C84268.pdf" H 8000 5250 50  0001 C CNN
+F 4 "Yellow 586~595nm 0603 Light Emitting Diodes (LED) RoHS" H 8000 5250 50  0001 C CNN "Description"
+F 5 "C84268" H 8000 5250 50  0001 C CNN "LCSC Part #"
+F 6 "Foshan NationStar Optoelectronics" H 8000 5250 50  0001 C CNN "Manufacturer"
+F 7 "15mA" H 8000 5250 50  0001 C CNN "Maximum Value"
+F 8 "KT-0603R" H 8000 5250 50  0001 C CNN "Mfr.Part #"
+F 9 "0603" H 8000 5250 50  0001 C CNN "Package Reference"
+	1    8000 5250
+	0    -1   -1   0
+$EndComp
 $EndSCHEMATC

Commit message: Rev 2 completed, todo check all and remove not needed filed
Parts:
- removed SW602: RST, Button_Switch_SMD:SW_SPST_EVQPE1, symbol Switch:SW_Push
- added SW502: RST, Button_Switch_SMD:SW_SPST_CK_RS282G05A3, symbol Switch:SW_Push
- C501: renamed from C601; Description 100nF ±10% 50V X7R 0603 Multilayer Ceramic Capacitors MLCC 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 -> (none); LCSC (none) -> C14663; LCSC Part # C478888 -> (none); Manufacturer TORCH -> (none); Mfr.Part # C0603B104K500NT -> (none)
- C502: renamed from C602; footprint Capacitor_SMD:C_0603_1608Metric_Pad1.08x0.95mm_HandSolder -> Capacitor_SMD:C_1206_3216Metric_Pad1.33x1.80mm_HandSolder; Description 47uF ±20% 6.3V X5R 0603 Multilayer Ceramic Capacitors MLCC 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 -> (none); LCSC (none) -> C96123; LCSC Part # C140782 -> (none); Manufacturer Murata Electronics -> (none); Maximum Value 6.3V -> 10V; Mfr.Part # GRM188R60J476ME15D -> (none); Package Reference 0603 -> 1206
- D501: renamed from D601; Description Yellow 586~595nm 0603 Light Emitting Diodes (LED) RoHS -> Blue; LCSC (none) -> C72041; LCSC Part # C84268 -> (none); Manufacturer Foshan NationStar Optoelectronics -> (none); Mfr.Part # KT-0603R -> (none)
- D502: renamed from D602; Description Yellow 586~595nm 0603 Light Emitting Diodes (LED) RoHS -> Blue; LCSC (none) -> C72041; LCSC Part # C84268 -> (none); Manufacturer Foshan NationStar Optoelectronics -> (none); Mfr.Part # KT-0603R -> (none)
- J501: renamed from J601; Description - -> (none); LCSC Part # - -> (none); Manufacturer - -> (none); Maximum Value - -> (none); Mfr.Part # - -> (none)
- JP501: renamed from JP601; Description - -> (none); LCSC Part # - -> (none); Manufacturer - -> (none); Maximum Value - -> (none); Mfr.Part # - -> (none)
- R501: renamed from R601; Description 10kΩ ±5% 0.1W ±100ppm/℃ 0603 Chip Resistor - Surface Mount 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 -> (none); LCSC (none) -> C25804; LCSC Part # C15401 -> (none); Manufacturer UNI-ROYAL(Uniroyal Elec) -> (none); Mfr.Part # 0603WAJ0103T5E -> (none)
- R502: renamed from R602; Description 10kΩ ±5% 0.1W ±100ppm/℃ 0603 Chip Resistor - Surface Mount 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 -> (none); LCSC (none) -> C25804; LCSC Part # C15401 -> (none); Manufacturer UNI-ROYAL(Uniroyal Elec) -> (none); Mfr.Part # 0603WAJ0103T5E -> (none)
- R503: renamed from R603; Description 10kΩ ±5% 0.1W ±100ppm/℃ 0603 Chip Resistor - Surface Mount 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 -> (none); LCSC (none) -> C25804; LCSC Part # C15401 -> (none); Manufacturer UNI-ROYAL(Uniroyal Elec) -> (none); Mfr.Part # 0603WAJ0103T5E -> (none)
- R504: renamed from R604; value 80 -> 15; footprint Resistor_SMD:R_0603_1608Metric_Pad0.98x0.95mm_HandSolder -> Resistor_SMD:R_0805_2012Metric_Pad1.20x1.40mm_HandSolder; Description 80.6Ω ±1% 0.1W ±100ppm/℃ 0603 Chip Resistor - Surface Mount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 -> (none); LCSC (none) -> C17480; LCSC Part # C202954 -> (none); Manufacturer BOURNS -> (none); Mfr.Part # CR0603-FX-80R6ELF -> (none); Package Reference 0603 -> 0805
- R505: renamed from R605; Description 10kΩ ±5% 0.1W ±100ppm/℃ 0603 Chip Resistor - Surface Mount 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 -> (none); LCSC (none) -> C25804; LCSC Part # C15401 -> (none); Manufacturer UNI-ROYAL(Uniroyal Elec) -> (none); Mfr.Part # 0603WAJ0103T5E -> (none)
- R506: renamed from R606; Description 10kΩ ±5% 0.1W ±100ppm/℃ 0603 Chip Resistor - Surface Mount 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 -> (none); LCSC (none) -> C25804; LCSC Part # C15401 -> (none); Manufacturer UNI-ROYAL(Uniroyal Elec) -> (none); Mfr.Part # 0603WAJ0103T5E -> (none)
- R507: renamed from R607; value 80 -> 15; footprint Resistor_SMD:R_0603_1608Metric_Pad0.98x0.95mm_HandSolder -> Resistor_SMD:R_0805_2012Metric_Pad1.20x1.40mm_HandSolder; Description 80.6Ω ±1% 0.1W ±100ppm/℃ 0603 Chip Resistor - Surface Mount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 -> (none); LCSC (none) -> C17480; LCSC Part # C202954 -> (none); Manufacturer BOURNS -> (none); Mfr.Part # CR0603-FX-80R6ELF -> (none); Package Reference 0603 -> 0805
- SW501: renamed from SW601; footprint Button_Switch_SMD:SW_SPST_EVQPE1 -> Button_Switch_SMD:SW_SPST_CK_RS282G05A3; Description SMD Tactile Switches RoHS -> (none); LCSC (none) -> C319365; LCSC (alt) (none) -> C398053; LCSC Part # C557591 -> (none); Manufacturer SHOU HAN -> (none); Maximum Value Pad |<- 3.4mm ->| [2.1x2mm] -> (none); Mfr.Part # TS342A2P-WZ -> (none); Package Reference 3.95x2.9x2mm -> 6.1x3.7x2.5mm
- U501: renamed from U601; LCSC (none) -> C82891; LCSC Part # C82891 -> (none); Manufacturer Ai-Thinker -> (none); Mfr.Part # ESP-12F(ESP8266MOD) -> (none)
Connections:
- net GND: now also SW502.1
- net ~RST: now also SW502.2
