File: pcb/Electra/Electra.sch (KiCad schematic (older format))
At the start: 2 parts, among them J101 Conn_01x04_Female, J102 Conn_01x07_Female

Commit message: PCB Ver 1 completed (TODO: Check)
Parts:
- removed J101: Conn_01x04_Female, Connector_PinHeader_2.54mm:PinHeader_1x04_P2.54mm_Vertical, symbol Connector:Conn_01x04_Female
- removed J102: Conn_01x07_Female, Connector_PinHeader_2.54mm:PinHeader_1x06_P2.54mm_Vertical, symbol Connector:Conn_01x07_Female
- added J101: Conn_01x06_Female, Connector_PinHeader_2.54mm:PinHeader_1x06_P2.54mm_Vertical, symbol Connector:Conn_01x06_Female
- added J102: Conn_01x04_Female, Connector_PinHeader_2.54mm:PinHeader_1x04_P2.54mm_Vertical, symbol Connector:Conn_01x04_Female
Connections:
- net +3V3: now also J101.5 (Pin_5), J102.4 (Pin_4)
- net GND: now also J101.6 (Pin_6), J102.3 (Pin_3)
- net L-SDA: now also J101.4 (Pin_4)
- net L-SDL: now also J101.3 (Pin_3)
- new net RX: J102.2 (Pin_2)
- new net TX: J102.1 (Pin_1)
- no-connect marks 5 -> 3
Other:
- note added: "(RX Led)"
- note added: "(TX Led)"
- note added: "ADC"
- note added: "HC06"
- note added: "RF433Mhz"
- note removed: "External RF433Mhz module"
- note removed: "RX Led"
- note removed: "TX Led"
Changed lines of the file:
@@
 $Descr A4 11693 8268
 encoding utf-8
-Sheet 1 7
+Sheet 1 8
 Title "Electra Project"
 Date "2021-03-21"
@@
 $EndDescr
 $Sheet
-S 4250 5900 2250 1300
+S 3500 5900 2250 1300
 U 60781751
 F0 "Power" 50
@@
 $EndSheet
 $Bitmap
-Pos 6300 3100
+Pos 6150 3100
 Scale 1.000000
 Data
@@
 	9550 1400 9450 1400
 Wire Wire Line
-	8750 3000 8850 3000
+	8600 3000 8700 3000
 Wire Wire Line
-	8750 2450 8850 2450
+	8600 2450 8700 2450
 Wire Wire Line
-	3350 4050 3200 4050
+	3200 4050 3050 4050
 Wire Wire Line
-	3350 3350 3200 3350
+	3200 3350 3050 3350
 Wire Wire Line
-	3350 2600 3200 2600
+	3200 2600 2450 2600
 Wire Wire Line
-	3350 1900 3200 1900
+	3200 1900 3050 1900
 Wire Wire Line
 	9500 5150 9400 5150
@@
 Text Label 9450 1400 2    50   ~ 10
 Relay1
-Text Label 8850 3000 0    50   ~ 10
+Text Label 8700 3000 0    50   ~ 10
 L-SDA
-Text Label 8850 2450 0    50   ~ 10
+Text Label 8700 2450 0    50   ~ 10
 L-SDL
-Text Label 3200 4050 2    50   ~ 10
+Text Label 3050 4050 2    50   ~ 10
 Relay1
-Text Label 3200 3350 2    50   ~ 10
+Text Label 3050 3350 2    50   ~ 10
 Switch1
-Text Label 3200 2600 2    50   ~ 10
-RF433Mhz
-Text Label 3200 1900 2    50   ~ 10
+Text Label 3050 1900 2    50   ~ 10
 Switch2
-Wire Wire Line
-	1700 6000 1600 6000
-Wire Wire Line
-	1700 5900 1600 5900
-Text Label 1600 6000 2    50   ~ 10
-L-SDA
-Text Label 1600 5900 2    50   ~ 10
-L-SDL
-Text Label 8850 4850 0    50   ~ 10
+Text Label 8700 4850 0    50   ~ 10
 Relay2
 Wire Wire Line
-	8750 4850 8850 4850
+	8600 4850 8700 4850
 $Sheet
-S 3350 950  5400 4200
+S 3200 950  5400 4200
 U 606FF326
 F0 "ESP8266" 50
 F1 "ESP8266.sch" 50
-F2 "GPIO15" B R 8750 4850 50
-F3 "GPIO4" B R 8750 3000 50
-F4 "GPIO5" B R 8750 2450 50
-F5 "GPIO12" B L 3350 3350 50
-F6 "GPIO13" B L 3350 4050 50
-F7 "GPIO14" B L 3350 2600 50
-F8 "GPIO16" B L 3350 1900 50
-F9 "GPIO2" B R 8750 4250 50
-F10 "GPIO3" B R 8750 1900 50
-F11 "GPIO1" B R 8750 1400 50
-F12 "GPIO0" B R 8750 3650 50
-F13 "GPIO10" B L 3350 4700 50
-F14 "ADC" B L 3350 1350 50
+F2 "GPIO15" B R 8600 4850 50
+F3 "GPIO4" B R 8600 3000 50
+F4 "GPIO5" B R 8600 2450 50
+F5 "GPIO12" B L 3200 3350 50
+F6 "GPIO13" B L 3200 4050 50
+F7 "GPIO14" B L 3200 2600 50
+F8 "GPIO16" B L 3200 1900 50
+F9 "GPIO2" B R 8600 4250 50
+F10 "GPIO3" B R 8600 1900 50
+F11 "GPIO1" B R 8600 1400 50
+F12 "GPIO0" B R 8600 3650 50
+F13 "GPIO10" B L 3200 4700 50
+F14 "ADC" B L 3200 1350 50
+$EndSheet
+NoConn ~ 3200 4700
+Text Notes 1200 5400 0    50   ~ 0
+External RTC module
+Text Notes 8200 1300 0    50   ~ 0
+(TX Led)
+Text Notes 8200 1800 0    50   ~ 0
+(RX Led)
+Text Notes 8600 3800 0    50   ~ 0
+Flash Button
+Text Notes 4000 6550 0    50   ~ 0
+USB or 8-28V DC Input  circuit
+$Sheet
+S 1150 1000 1300 700
+U 60D319D8
+F0 "ADC-logic" 50
+F1 "ADC-logic.sch" 50
+F2 "output" O R 2450 1350 50
 $EndSheet
-NoConn ~ 3350 4700
+Wire Wire Line
+	2450 1350 3200 1350
+Wire Wire Line
+	8600 1400 8650 1400
+Wire Wire Line
+	8600 1900 8650 1900
+Text Label 8650 1400 0    50   ~ 0
+TX
+Text Label 8650 1900 0    50   ~ 0
+RX
+Wire Wire Line
+	7650 5750 7550 5750
+Wire Wire Line
+	7650 5850 7550 5850
+Wire Wire Line
+	7650 5950 7550 5950
+Wire Wire Line
+	7650 6050 7550 6050
+Text Label 7550 5750 2    50   ~ 0
+TX
 $Comp
-L Connector:Conn_01x07_Female J102
-U 1 1 60C78016
-P 1900 5900
-F 0 "J102" H 1928 5926 50  0000 L CNN
-F 1 "Conn_01x07_Female" H 1928 5835 50  0000 L CNN
-F 2 "Connector_PinHeader_2.54mm:PinHeader_1x06_P2.54mm_Vertical" H 1900 5900 50  0001 C CNN
-F 3 "~" H 1900 5900 50  0001 C CNN
-	1    1900 5900
-	1    0    0    -1
+L power:GND #PWR0103
+U 1 1 605BF872
+P 7550 5950
+F 0 "#PWR0103" H 7550 5700 50  0001 C CNN
+F 1 "GND" H 7555 5777 50  0000 C CNN
+F 2 "" H 7550 5950 50  0001 C CNN
+F 3 "" H 7550 5950 50  0001 C CNN
+	1    7550 5950
+	0    1    1    0
 $EndComp
 $Comp
-L power:GND #PWR0104
+L power:+3V3 #PWR0104
+U 1 1 605C0C61
+P 7550 6050
+F 0 "#PWR0104" H 7550 5900 50  0001 C CNN
+F 1 "+3V3" V 7450 6050 50  0000 L CNN
+F 2 "" H 7550 6050 50  0001 C CNN
+F 3 "" H 7550 6050 50  0001 C CNN
+	1    7550 6050
+	0    -1   -1   0
+$EndComp
+Text Label 7550 5850 2    50   ~ 0
+RX
+Text Notes 7600 5550 0    50   ~ 0
+HC06
+$Sheet
+S 1150 2300 1300 650
+U 605DAAEC
+F0 "RF433Hz-Receiver" 50
+F1 "RF433Hz-Receiver.sch" 50
+F2 "output" O R 2450 2600 50
+$EndSheet
+Text Notes 2600 2600 0    50   ~ 0
+RF433Mhz
+Text Notes 2900 1350 0    50   ~ 0
+ADC
+Wire Wire Line
+	1600 5850 1500 5850
+Wire Wire Line
+	1600 5750 1500 5750
+Text Label 1500 5850 2    50   ~ 10
+L-SDA
+Text Label 1500 5750 2    50   ~ 10
+L-SDL
+$Comp
+L power:GND #PWR0102
 U 1 1 60C78A09
-P 1450 6300
-F 0 "#PWR0104" H 1450 6050 50  0001 C CNN
-F 1 "GND" H 1455 6127 50  0000 C CNN
-F 2 "" H 1450 6300 50  0001 C CNN
-F 3 "" H 1450 6300 50  0001 C CNN
-	1    1450 6300
+P 1350 6150
+F 0 "#PWR0102" H 1350 5900 50  0001 C CNN
+F 1 "GND" H 1355 5977 50  0000 C CNN
+F 2 "" H 1350 6150 50  0001 C CNN
+F 3 "" H 1350 6150 50  0001 C CNN
+	1    1350 6150
 	1    0    0    -1
 $EndComp
@@
 L power:+3V3 #PWR0101
 U 1 1 60C78E20
-P 1150 5950
-F 0 "#PWR0101" H 1150 5800 50  0001 C CNN
-F 1 "+3V3" V 1165 6078 50  0000 L CNN
-F 2 "" H 1150 5950 50  0001 C CNN
-F 3 "" H 1150 5950 50  0001 C CNN
-	1    1150 5950
+P 1050 5800
+F 0 "#PWR0101" H 1050 5650 50  0001 C CNN
+F 1 "+3V3" V 1065 5928 50  0000 L CNN
+F 2 "" H 1050 5800 50  0001 C CNN
+F 3 "" H 1050 5800 50  0001 C CNN
+	1    1050 5800
 	1    0    0    -1
 $EndComp
 Wire Wire Line
-	1700 6200 1450 6200
+	1600 6050 1350 6050
 Wire Wire Line
-	1450 6200 1450 6300
-NoConn ~ 1700 5600
-NoConn ~ 1700 5700
-NoConn ~ 1700 5800
+	1350 6050 1350 6150
 Wire Wire Line
-	1150 6100 1700 6100
+	1050 5950 1600 5950
 Wire Wire Line
-	1150 5950 1150 6100
-Text Notes 1200 5400 0    50   ~ 0
-External RTC module
+	1050 5800 1050 5950
+NoConn ~ 1600 5650
+NoConn ~ 1600 5550
 $Comp
-L Connector:Conn_01x04_Female J101
-U 1 1 60C81EF7
-P 1600 3650
-F 0 "J101" H 1628 3626 50  0000 L CNN
-F 1 "Conn_01x04_Female" H 1628 3535 50  0000 L CNN
-F 2 "Connector_PinHeader_2.54mm:PinHeader_1x04_P2.54mm_Vertical" H 1600 3650 50  0001 C CNN
-F 3 "~" H 1600 3650 50  0001 C CNN
-	1    1600 3650
+L Connector:Conn_01x04_Female J102
+U 1 1 605BB00E
+P 7850 5850
+F 0 "J102" H 7878 5826 50  0000 L CNN
+F 1 "Conn_01x04_Female" H 7878 5735 50  0000 L CNN
+F 2 "Connector_PinHeader_2.54mm:PinHeader_1x04_P2.54mm_Vertical" H 7850 5850 50  0001 C CNN
+F 3 "-" H 7850 5850 50  0001 C CNN
+F 4 "-" H 7850 5850 50  0001 C CNN "Mfr.Part #"
+F 5 "2.54mm" H 7850 5850 50  0001 C CNN "Package Reference"
+F 6 "-" H 7850 5850 50  0001 C CNN "Description"
+F 7 "-" H 7850 5850 50  0001 C CNN "LCSC Part #"
+F 8 "-" H 7850 5850 50  0001 C CNN "Manufacturer"
+F 9 "-" H 7850 5850 50  0001 C CNN "Maximum Value"
+	1    7850 5850
 	1    0    0    -1
 $EndComp
 $Comp
-L power:GND #PWR0103
-U 1 1 60C82480
-P 1250 3900
-F 0 "#PWR0103" H 1250 3650 50  0001 C CNN
-F 1 "GND" H 1255 3727 50  0000 C CNN
-F 2 "" H 1250 3900 50  0001 C CNN
-F 3 "" H 1250 3900 50  0001 C CNN
-	1    1250 3900
+L Connector:Conn_01x06_Female J101
+U 1 1 60626341
+P 1800 5750
+F 0 "J101" H 1828 5726 50  0000 L CNN
+F 1 "Conn_01x06_Female" H 1828 5635 50  0000 L CNN
+F 2 "Connector_PinHeader_2.54mm:PinHeader_1x06_P2.54mm_Vertical" H 1800 5750 50  0001 C CNN
+F 3 "~" H 1800 5750 50  0001 C CNN
+F 4 "-" H 1800 5750 50  0001 C CNN "Description"
+F 5 "-" H 1800 5750 50  0001 C CNN "LCSC Part #"
+F 6 "-" H 1800 5750 50  0001 C CNN "Manufacturer"
+F 7 "-" H 1800 5750 50  0001 C CNN "Maximum Value"
+F 8 "-" H 1800 5750 50  0001 C CNN "Mfr.Part #"
+F 9 "-" H 1800 5750 50  0001 C CNN "Package Reference"
+	1    1800 5750
 	1    0    0    -1
 $EndComp
-$Comp
-L power:+5V #PWR0102
-U 1 1 60C82996
-P 1250 3500
-F 0 "#PWR0102" H 1250 3350 50  0001 C CNN
-F 1 "+5V" H 1265 3673 50  0000 C CNN
-F 2 "" H 1250 3500 50  0001 C CNN
-F 3 "" H 1250 3500 50  0001 C CNN
-	1    1250 3500
-	1    0    0    -1
-$EndComp
-Text Label 1150 3650 2    50   ~ 10
-RF433Mhz
-Wire Wire Line
-	1400 3850 1250 3850
-Wire Wire Line
-	1250 3850 1250 3900
-Wire Wire Line
-	1150 3650 1400 3650
-Wire Wire Line
-	1400 3550 1250 3550
-Wire Wire Line
-	1250 3550 1250 3500
-Text Notes 1450 3400 0    50   ~ 0
-External RF433Mhz module
-NoConn ~ 1400 3750
-Text Notes 8800 1350 0    50   ~ 0
-TX Led
-Text Notes 8800 1800 0    50   ~ 0
-RX Led
-Text Notes 8750 3800 0    50   ~ 0
-Flash Button
-Text Notes 4750 6550 0    50   ~ 0
-USB or 8-28V DC Input  circuit
-$Sheet
-S 1150 1000 1300 700
-U 60D319D8
-F0 "ADC-logic" 50
-F1 "ADC-logic.sch" 50
-F2 "output" O R 2450 1350 50
-$EndSheet
-Wire Wire Line
-	2450 1350 3350 1350
 $EndSCHEMATC

Commit message: PCB completed (added silkscreen more)
Parts:
- J101: value Conn_01x06_Female -> RTC
- J102: value Conn_01x04_Female -> UART

Commit message: Rev 2 completed, todo check all and remove not needed filed
Parts:
- added J101: Extra1, Connector_PinHeader_2.54mm:PinHeader_1x03_P2.54mm_Vertical, symbol Connector:Conn_01x03_Female
- added J103: Extra2, Connector_PinHeader_2.54mm:PinHeader_1x03_P2.54mm_Vertical, symbol Connector:Conn_01x03_Female
- J102: renamed from J101; Description - -> (none); LCSC Part # - -> (none); Manufacturer - -> (none); Mfr.Part # - -> (none); Package Reference - -> 2.54mm
- J104: renamed from J102; Description - -> (none); LCSC Part # - -> (none); Manufacturer - -> (none); Mfr.Part # - -> (none)
Connections:
- net +3V3: now also J101.1 (Pin_1), J103.1 (Pin_1)
- net GND: now also J101.3 (Pin_3), J103.3 (Pin_3)
- new net Extra1: J101.2 (Pin_2)
- new net Extra2: J103.2 (Pin_2)
- no-connect marks 3 -> 2
Other:
- note added: "Maybe button footprint fix"
- moved on the sheet: J102, J104

Commit message: IMPORTANT! REV 2 completed! Send to fabrication
Other:
- note added: "USB or 7-12V DC Input circuit"
- note removed: "USB or 8-28V DC Input circuit"
Changed lines of the file:
@@
 Flash Button
 Text Notes 4950 6850 0    50   ~ 0
-USB or 8-28V DC Input  circuit
+USB or 7-12V DC Input  circuit
 $Sheet
 S 1150 1000 1300 700

Commit message: Minor fixes on schematic and pcb fix bjt netlist + ac main voltage to both sides (Rev 2.1)
Other:
- note added: "ONLY as Output"
Changed lines of the file:
@@
 Sheet 1 8
 Title "Electra Project"
-Date "2021-04-01"
-Rev "2.0"
+Date "2021-05-04"
+Rev "2.1"
 Comp "Grehasopt"
 Comment1 "https://github.com/Grehasopt/Electra"
@@
 Text Label 2100 4450 2    50   ~ 10
 Extra2
+Text Notes 2050 5050 0    50   ~ 0
+ONLY as Output
 $EndSCHEMATC
