File: pcb/Electra/Power.sch (KiCad schematic (older format))
At the start: 26 parts, among them J201 8-28VIn, J202 USB_B_Micro, J203 Enable VIn, U201 AMS1117-3.3, U202 TPS54202DDCR

Commit message: PCB Ver 1 completed (TODO: Check)
Parts:
- C201, C205, C206: Manufacturer (none) -> Taiyo Yuden
- C202, C204: Manufacturer (none) -> YAGEO
- C203, C208: Manufacturer (none) -> Honor Elec
- C207: Manufacturer (none) -> FH(Guangdong Fenghua Advanced Tech)
- D201: Manufacturer (none) -> MDD(Microdiode Electronics)
- D202: Manufacturer (none) -> Everlight Elec
- J201: Manufacturer (none) -> BOOMELE(Boom Precision Elec)
- J202: Manufacturer (none) -> Jing Extension of the Electronic Co.
- J203: Manufacturer (none) -> Ckmtw(Shenzhen Cankemeng)
- L201: Manufacturer (none) -> Sumida
- R201, R202, R205, R206: Manufacturer (none) -> UNI-ROYAL(Uniroyal Elec)
- R203: footprint Resistor_SMD:R_0201_0603Metric_Pad0.64x0.40mm_HandSolder -> Resistor_SMD:R_0603_1608Metric_Pad0.98x0.95mm_HandSolder; Manufacturer (none) -> Ever Ohms Tech
- R204: Manufacturer (none) -> Walsin Tech Corp
Changed lines of the file:
@@
 $Descr A4 11693 8268
 encoding utf-8
-Sheet 2 7
+Sheet 2 8
 Title "Electra Project"
 Date "2021-03-21"
@@
 F 7 "C23194" H 5100 2350 50  0001 C CNN "LCSC Part #"
 F 8 "0603WAF5113T5E" H 5100 2350 50  0001 C CNN "Mfr.Part #"
+F 9 "UNI-ROYAL(Uniroyal Elec)" H 5100 2350 50  0001 C CNN "Manufacturer"
 	1    5100 2350
 	1    0    0    -1
@@
 F 7 "C124375" H 8900 2200 50  0001 C CNN "Mfr.Part #"
 F 8 "2.54mm" H 8900 2200 50  0001 C CNN "Package Reference"
+F 9 "Ckmtw(Shenzhen Cankemeng)" H 8900 2200 50  0001 C CNN "Manufacturer"
 	1    8900 2200
 	1    0    0    -1
@@
 F 7 "RVT1A101M0505" H 6350 5250 50  0001 C CNN "Mfr.Part #"
 F 8 "SMD,5x5.4mm" H 6350 5250 50  0001 C CNN "Package Reference"
+F 9 "Honor Elec" H 6350 5250 50  0001 C CNN "Manufacturer"
 	1    6350 5250
 	1    0    0    -1
@@
 F 7 "RVT1A101M0505" H 9900 2750 50  0001 C CNN "Mfr.Part #"
 F 8 "SMD,5x5.4mm" H 9900 2750 50  0001 C CNN "Package Reference"
+F 9 "Honor Elec" H 9900 2750 50  0001 C CNN "Manufacturer"
 	1    9900 2750
 	1    0    0    -1
@@
 F 7 "19-217/GHC-YR1S2/3T" H 7000 5350 50  0001 C CNN "Mfr.Part #"
 F 8 "0603" H 7000 5350 50  0001 C CNN "Package Reference"
+F 9 "Everlight Elec" H 7000 5350 50  0001 C CNN "Manufacturer"
 	1    7000 5350
 	0    -1   -1   0
-$EndComp
-$Comp
-L Device:R R203
-U 1 1 60BE5E4B
-P 7000 5050
-F 0 "R203" V 6900 5150 50  0000 R CNN
-F 1 "80" V 7000 5100 50  0000 R CNN
-F 2 "Resistor_SMD:R_0201_0603Metric_Pad0.64x0.40mm_HandSolder" V 6930 5050 50  0001 C CNN
-F 3 "https://datasheet.lcsc.com/szlcsc/1912111437_Ever-Ohms-Tech-CR0603F80R6P05_C429015.pdf" H 7000 5050 50  0001 C CNN
-F 4 "0603" H 7000 5050 50  0001 C CNN "Package Reference"
-F 5 "80.6Ω ±1% 0.1W ±100ppm/℃ 0603 Chip Resistor - Surface Mount RoHS" H 7000 5050 50  0001 C CNN "Description"
-F 6 "C429015" H 7000 5050 50  0001 C CNN "LCSC Part #"
-F 7 "0.1W" H 7000 5050 50  0001 C CNN "Maximum Value"
-F 8 "CR0603F80R6P05" H 7000 5050 50  0001 C CNN "Mfr.Part #"
-	1    7000 5050
-	-1   0    0    1
 $EndComp
 Wire Wire Line
@@
 F 7 "920-E52A2021S10100" H 4100 5000 50  0001 C CNN "Mfr.Part #"
 F 8 "SMD" H 4100 5000 50  0001 C CNN "Package Reference"
+F 9 "Jing Extension of the Electronic Co." H 4100 5000 50  0001 C CNN "Manufacturer"
 	1    4100 5000
 	1    0    0    -1
@@
 F 7 "C225048" H 7000 2200 50  0001 C CNN "LCSC Part #"
 F 8 "CDRH104RNP-150NC" H 7000 2200 50  0001 C CNN "Mfr.Part #"
+F 9 "Sumida" H 7000 2200 50  0001 C CNN "Manufacturer"
 	1    7000 2200
 	0    -1   -1   0
@@
 F 7 "C25952" H 8250 3150 50  0001 C CNN "LCSC Part #"
 F 8 "0603WAF1332T5E" H 8250 3150 50  0001 C CNN "Mfr.Part #"
+F 9 "UNI-ROYAL(Uniroyal Elec)" H 8250 3150 50  0001 C CNN "Manufacturer"
 	1    8250 3150
 	1    0    0    -1
@@
 F 7 "C15458" H 8250 2750 50  0001 C CNN "LCSC Part #"
 F 8 "0603WAJ0104T5E" H 8250 2750 50  0001 C CNN "Mfr.Part #"
+F 9 "UNI-ROYAL(Uniroyal Elec)" H 8250 2750 50  0001 C CNN "Manufacturer"
 	1    8250 2750
 	1    0    0    -1
@@
 F 7 "C163926" H 8250 2350 50  0001 C CNN "LCSC Part #"
 F 8 "WR06X49R9FTL" H 8250 2350 50  0001 C CNN "Mfr.Part #"
+F 9 "Walsin Tech Corp" H 8250 2350 50  0001 C CNN "Manufacturer"
 	1    8250 2350
 	1    0    0    -1
@@
 F 7 "C16840" H 5100 2900 50  0001 C CNN "LCSC Part #"
 F 8 "0603WAF1053T5E" H 5100 2900 50  0001 C CNN "Mfr.Part #"
+F 9 "UNI-ROYAL(Uniroyal Elec)" H 5100 2900 50  0001 C CNN "Manufacturer"
 	1    5100 2900
 	1    0    0    -1
@@
 F 7 "C337451" H 7700 2350 50  0001 C CNN "LCSC Part #"
 F 8 "TMK325B7226KM-PR" H 7700 2350 50  0001 C CNN "Mfr.Part #"
+F 9 "Taiyo Yuden" H 7700 2350 50  0001 C CNN "Manufacturer"
 	1    7700 2350
 	-1   0    0    1
@@
 F 7 "C1681" H 8000 2750 50  0001 C CNN "LCSC Part #"
 F 8 "0603CG750J500NT" H 8000 2750 50  0001 C CNN "Mfr.Part #"
+F 9 "FH(Guangdong Fenghua Advanced Tech)" H 8000 2750 50  0001 C CNN "Manufacturer"
 	1    8000 2750
 	-1   0    0    1
@@
 F 7 "C337451" H 7300 2350 50  0001 C CNN "LCSC Part #"
 F 8 "TMK325B7226KM-PR" H 7300 2350 50  0001 C CNN "Mfr.Part #"
+F 9 "Taiyo Yuden" H 7300 2350 50  0001 C CNN "Manufacturer"
 	1    7300 2350
 	-1   0    0    1
@@
 F 7 "C92490" H 6450 2000 50  0001 C CNN "LCSC Part #"
 F 8 "CC0603KRX7R8BB104" H 6450 2000 50  0001 C CNN "Mfr.Part #"
+F 9 "YAGEO" H 6450 2000 50  0001 C CNN "Manufacturer"
 	1    6450 2000
 	0    1    1    0
@@
 F 7 "C92490" H 4550 2600 50  0001 C CNN "LCSC Part #"
 F 8 "CC0603KRX7R8BB104" H 4550 2600 50  0001 C CNN "Mfr.Part #"
+F 9 "YAGEO" H 4550 2600 50  0001 C CNN "Manufacturer"
 	1    4550 2600
 	1    0    0    -1
@@
 F 7 "C92799" H 4150 2600 50  0001 C CNN "LCSC Part #"
 F 8 "GMK325BJ106KN-T" H 4150 2600 50  0001 C CNN "Mfr.Part #"
+F 9 "Taiyo Yuden" H 4150 2600 50  0001 C CNN "Manufacturer"
 	1    4150 2600
 	1    0    0    -1
@@
 F 7 "S2M" H 3250 2100 50  0001 C CNN "Mfr.Part #"
 F 8 " SMA(DO-214AC)" H 3250 2100 50  0001 C CNN "Package Reference"
+F 9 "MDD(Microdiode Electronics)" H 3250 2100 50  0001 C CNN "Manufacturer"
 	1    3250 2100
 	1    0    0    -1
@@
 F 7 "DC-005 5.5-2.0MM" H 1750 2200 50  0001 C CNN "Mfr.Part #"
 F 8 "-" H 1750 2200 50  0001 C CNN "Package Reference"
+F 9 "BOOMELE(Boom Precision Elec)" H 1750 2200 50  0001 C CNN "Manufacturer"
 	1    1750 2200
 	1    0    0    -1
 $EndComp
+$Comp
+L Device:R R203
+U 1 1 60BE5E4B
+P 7000 5050
+F 0 "R203" V 6900 5150 50  0000 R CNN
+F 1 "80" V 7000 5100 50  0000 R CNN
+F 2 "Resistor_SMD:R_0603_1608Metric_Pad0.98x0.95mm_HandSolder" V 6930 5050 50  0001 C CNN
+F 3 "https://datasheet.lcsc.com/szlcsc/1912111437_Ever-Ohms-Tech-CR0603F80R6P05_C429015.pdf" H 7000 5050 50  0001 C CNN
+F 4 "0603" H 7000 5050 50  0001 C CNN "Package Reference"
+F 5 "80.6Ω ±1% 0.1W ±100ppm/℃ 0603 Chip Resistor - Surface Mount RoHS" H 7000 5050 50  0001 C CNN "Description"
+F 6 "C429015" H 7000 5050 50  0001 C CNN "LCSC Part #"
+F 7 "0.1W" H 7000 5050 50  0001 C CNN "Maximum Value"
+F 8 "CR0603F80R6P05" H 7000 5050 50  0001 C CNN "Mfr.Part #"
+F 9 "Ever Ohms Tech" H 7000 5050 50  0001 C CNN "Manufacturer"
+	1    7000 5050
+	-1   0    0    1
+$EndComp
 $EndSCHEMATC

Commit message: PCB completed (added silkscreen more)
Parts:
- D202: value Power Led -> PWR
- J201: value 8-28VIn -> 8-28V
- J202: value USB_B_Micro -> USB
- R201, R202, R204, R205, R206: footprint Resistor_SMD:R_0201_0603Metric_Pad0.64x0.40mm_HandSolder -> Resistor_SMD:R_0603_1608Metric_Pad0.98x0.95mm_HandSolder
Changed lines of the file:
@@
 F 0 "R201" V 5000 2250 50  0000 L CNN
 F 1 "511K" V 5100 2250 50  0000 L CNN
-F 2 "Resistor_SMD:R_0201_0603Metric_Pad0.64x0.40mm_HandSolder" V 5030 2350 50  0001 C CNN
+F 2 "Resistor_SMD:R_0603_1608Metric_Pad0.98x0.95mm_HandSolder" V 5030 2350 50  0001 C CNN
 F 3 "https://datasheet.lcsc.com/szlcsc/1811081723_UNI-ROYAL-Uniroyal-Elec-0603WAF5113T5E_C23194.pdf" H 5100 2350 50  0001 C CNN
 F 4 "0.1W" H 5100 2350 50  0001 C CNN "Maximum Value"
@@
 P 7000 5350
 F 0 "D202" V 7050 5250 50  0000 R CNN
-F 1 "Power Led" V 6950 5250 50  0000 R CNN
+F 1 "PWR" V 6950 5250 50  0000 R CNN
 F 2 "LED_SMD:LED_0603_1608Metric_Pad1.05x0.95mm_HandSolder" H 7000 5350 50  0001 C CNN
 F 3 "https://datasheet.lcsc.com/szlcsc/1811101510_Everlight-Elec-19-217-GHC-YR1S2-3T_C72043.pdf" H 7000 5350 50  0001 C CNN
@@
 P 4100 5000
 F 0 "J202" H 4157 5467 50  0000 C CNN
-F 1 "USB_B_Micro" H 4157 5376 50  0000 C CNN
+F 1 "USB" H 4157 5376 50  0000 C CNN
 F 2 "Connector_USB:USB_Micro-B_Molex-105017-0001" H 4250 4950 50  0001 C CNN
 F 3 "https://datasheet.lcsc.com/szlcsc/2103051832_Jing-Extension-of-the-Electronic-Co-920-E52A2021S10100_C10418.pdf" H 4250 4950 50  0001 C CNN
@@
 F 0 "R206" V 8350 3050 50  0000 L CNN
 F 1 "13.3K" V 8250 3050 50  0000 L CNN
-F 2 "Resistor_SMD:R_0201_0603Metric_Pad0.64x0.40mm_HandSolder" V 8180 3150 50  0001 C CNN
+F 2 "Resistor_SMD:R_0603_1608Metric_Pad0.98x0.95mm_HandSolder" V 8180 3150 50  0001 C CNN
 F 3 "https://datasheet.lcsc.com/szlcsc/1811021221_UNI-ROYAL-Uniroyal-Elec-0603WAF1332T5E_C25952.pdf" H 8250 3150 50  0001 C CNN
 F 4 "0.1W" H 8250 3150 50  0001 C CNN "Maximum Value"
@@
 F 0 "R205" V 8350 2650 50  0000 L CNN
 F 1 "100K" V 8250 2650 50  0000 L CNN
-F 2 "Resistor_SMD:R_0201_0603Metric_Pad0.64x0.40mm_HandSolder" V 8180 2750 50  0001 C CNN
+F 2 "Resistor_SMD:R_0603_1608Metric_Pad0.98x0.95mm_HandSolder" V 8180 2750 50  0001 C CNN
 F 3 "https://datasheet.lcsc.com/szlcsc/1811081710_UNI-ROYAL-Uniroyal-Elec-0603WAJ0104T5E_C15458.pdf" H 8250 2750 50  0001 C CNN
 F 4 "0.1W" H 8250 2750 50  0001 C CNN "Maximum Value"
@@
 F 0 "R204" V 8350 2250 50  0000 L CNN
 F 1 "49.9" V 8250 2250 50  0000 L CNN
-F 2 "Resistor_SMD:R_0201_0603Metric_Pad0.64x0.40mm_HandSolder" V 8180 2350 50  0001 C CNN
+F 2 "Resistor_SMD:R_0603_1608Metric_Pad0.98x0.95mm_HandSolder" V 8180 2350 50  0001 C CNN
 F 3 "https://datasheet.lcsc.com/szlcsc/1811151149_Walsin-Tech-Corp-WR06X49R9FTL_C163926.pdf" H 8250 2350 50  0001 C CNN
 F 4 "0.1W" H 8250 2350 50  0001 C CNN "Maximum Value"
@@
 F 0 "R202" V 5000 2800 50  0000 L CNN
 F 1 "105K" V 5100 2800 50  0000 L CNN
-F 2 "Resistor_SMD:R_0201_0603Metric_Pad0.64x0.40mm_HandSolder" V 5030 2900 50  0001 C CNN
+F 2 "Resistor_SMD:R_0603_1608Metric_Pad0.98x0.95mm_HandSolder" V 5030 2900 50  0001 C CNN
 F 3 "https://datasheet.lcsc.com/szlcsc/1811151640_UNI-ROYAL-Uniroyal-Elec-0603WAF1053T5E_C16840.pdf" H 5100 2900 50  0001 C CNN
 F 4 "0.1W" H 5100 2900 50  0001 C CNN "Maximum Value"
@@
 P 1750 2200
 F 0 "J201" H 1750 2400 50  0000 C CNN
-F 1 "8-28VIn" H 1750 2000 50  0000 C CNN
+F 1 "8-28V" H 1750 2000 50  0000 C CNN
 F 2 "Connector_BarrelJack:BarrelJack_Horizontal" H 1800 2160 50  0001 C CNN
 F 3 "https://datasheet.lcsc.com/szlcsc/1811051112_BOOMELE-Boom-Precision-Elec-DC-005-5-5-2-0MM_C16214.pdf" H 1800 2160 50  0001 C CNN

Commit message: Rev 2 completed, todo check all and remove not needed filed
Parts:
- removed C201: 10uF, Capacitor_SMD:C_1210_3225Metric_Pad1.33x2.70mm_HandSolder, symbol Device:C
- removed C203, C208: 100uF, Capacitor_SMD:CP_Elec_5x5.4, symbol Device:CP
- removed C204: 0.1uF, Capacitor_SMD:C_0603_1608Metric_Pad1.08x0.95mm_HandSolder, symbol Device:C
- removed C205, C206: 22uF, Capacitor_SMD:C_1210_3225Metric_Pad1.33x2.70mm_HandSolder, symbol Device:C
- removed C207: 75pF, Capacitor_SMD:C_0603_1608Metric_Pad1.08x0.95mm_HandSolder, symbol Device:C
- removed D202: PWR, LED_SMD:LED_0603_1608Metric_Pad1.05x0.95mm_HandSolder, symbol Device:LED
- removed J201: 8-28V, Connector_BarrelJack:BarrelJack_Horizontal, symbol Connector:Barrel_Jack
- removed J202: USB, Connector_USB:USB_Micro-B_Molex-105017-0001, symbol Connector:USB_B_Micro
- removed J203: Enable VIn, Connector_PinHeader_2.54mm:PinHeader_2x01_P2.54mm_Vertical, symbol Connector_Generic:Conn_02x01
- removed L201: 15uH, Inductor_SMD:L_10.4x10.4_H4.8, symbol Device:L_Core_Iron_Small
- removed R202: 105K, Resistor_SMD:R_0603_1608Metric_Pad0.98x0.95mm_HandSolder, symbol Device:R
- removed R203: 80, Resistor_SMD:R_0603_1608Metric_Pad0.98x0.95mm_HandSolder, symbol Device:R
- removed R204: 49.9, Resistor_SMD:R_0603_1608Metric_Pad0.98x0.95mm_HandSolder, symbol Device:R
- removed R205: 100K, Resistor_SMD:R_0603_1608Metric_Pad0.98x0.95mm_HandSolder, symbol Device:R
- removed R206: 13.3K, Resistor_SMD:R_0603_1608Metric_Pad0.98x0.95mm_HandSolder, symbol Device:R
- removed U201: AMS1117-3.3, Package_TO_SOT_SMD:SOT-223-3_TabPin2, symbol Regulator_Linear:AMS1117-3.3
- removed U202: TPS54202DDCR, Package_TO_SOT_SMD:SOT-23-6, symbol Regulator_Switching:TPS54202DDC
- added C201, C204, C205: 100uF, Capacitor_SMD:CP_Elec_6.3x5.4, symbol Device:CP
- added C203: 10uF, Capacitor_SMD:C_0805_2012Metric_Pad1.18x1.45mm_HandSolder, symbol Device:C
- added D202, D203: 1A, Diode_SMD:D_SMA_Handsoldering, symbol pspice:DIODE
- added D204: PWR, LED_SMD:LED_0603_1608Metric_Pad1.05x0.95mm_HandSolder, symbol Device:LED
- added J201: USB, Connector_USB:USB_Micro-B_Molex-105017-0001, symbol Connector:USB_B_Micro
- added J202: 7-12V, Connector_BarrelJack:BarrelJack_Horizontal, symbol Connector:Barrel_Jack
- added JP201: Jumper_NC_Small, Jumper:SolderJumper-2_P1.3mm_Bridged_RoundedPad1.0x1.5mm, symbol Device:Jumper_NC_Small
- added U201: AMS1117-5.0, Package_TO_SOT_SMD:SOT-223-3_TabPin2, symbol Regulator_Linear:AMS1117-5.0
- added U202: AMS1117-3.3, Package_TO_SOT_SMD:SOT-223-3_TabPin2, symbol Regulator_Linear:AMS1117-3.3
- C202: value 0.1uF -> 10uF; footprint Capacitor_SMD:C_0603_1608Metric_Pad1.08x0.95mm_HandSolder -> Capacitor_SMD:C_0805_2012Metric_Pad1.18x1.45mm_HandSolder; Description 100nF ±10% 25V X7R 0603 Multilayer Ceramic Capacitors MLCC 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 -> (none); LCSC (none) -> C15850; LCSC Part # C92490 -> (none); Manufacturer YAGEO -> (none); Maximum Value 25V -> (none); Maximum value (none) -> 25V; Mfr.Part # CC0603KRX7R8BB104 -> (none); Package Reference 0603 -> (none)
- D201: value DIODE -> 1A; footprint Diode_SMD:D_SMA -> Diode_SMD:D_SMA_Handsoldering; Description 1kV 2A 1.1V @ 2A SMA(DO-214AC) Diodes - General Purpose RoHS -> (none); LCSC (none) -> C95872; LCSC Part # C18905 -> (none); Manufacturer MDD(Microdiode Electronics) -> (none); Maximum Value 2A -> 1A; Mfr.Part # S2M -> (none)
- R201: value 511K -> 82; Description 511kΩ ±1% 0.1W ±100ppm/℃ 0603 Chip Resistor - Surface Mount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 -> (none); LCSC (none) -> C23255; LCSC Part # C23194 -> (none); Manufacturer UNI-ROYAL(Uniroyal Elec) -> (none); Mfr.Part # 0603WAF5113T5E -> (none)
- TP201, TP202: Description - -> (none); LCSC Part # - -> (none); Manufacturer - -> (none); Mfr.Part # - -> (none)
- TP203: value 3V3 -> 5V; Description - -> (none); LCSC Part # - -> (none); Manufacturer - -> (none); Mfr.Part # - -> (none)
- TP204: value 5V -> 3V3; Description - -> (none); LCSC Part # - -> (none); Manufacturer - -> (none); Mfr.Part # - -> (none)
Connections:
- net +3V3: now also C202.1, R201.2, TP204.1, C204.1, U202.2 (VO); no longer TP203.1
- net +5V: now also TP203.1, C203.1, C205.1, D203.1 (K), JP201.2, U201.2 (VO); no longer TP204.1
- net +VDC: now also D202.1 (K), J202.1
- net GND: now also C201.2, C203.2, C204.2, C205.2, D204.1 (K), J201.5 (GND), J201.6 (Shield), J202.2, U201.1 (GND), U202.1 (GND)
- net at D201.2 (A), TP202.1: now also C201.1, D202.2 (A), D203.2 (A), U201.3 (VI), U202.3 (VI); no longer C202.1, R201.1
- new net: J201.1 (VBUS), JP201.1
- new net: D204.2 (A), R201.1
Other:
- note added: "3.3V 1A"
- note added: "5V 1A"
- note removed: "5V 2A"
