File: pcb/Electra/Reed Switches.sch (KiCad schematic (older format))
At the start: 4 parts, among them J501 Conn_01x02_Female, J502 Conn_01x02_Female

Commit message: PCB Ver 1 completed (TODO: Check)
Parts:
- J501, J502: Package Reference - -> 2.54mm 1x2
- R501, R502: Description https://datasheet.lcsc.com/szlcsc/1809140220_UNI-ROYAL-Unir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 -> 10kΩ ±5% 0.1W ±100ppm/℃ 0603 Chip Resistor - Surface Mount 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
Changed lines of the file:
@@
 $Descr A4 11693 8268
 encoding utf-8
-Sheet 5 7
+Sheet 5 8
 Title "Electra Project"
 Date "2021-03-21"
@@
 F 2 "Resistor_SMD:R_0603_1608Metric_Pad0.98x0.95mm_HandSolder" V 3580 3300 50  0001 C CNN
 F 3 "https://datasheet.lcsc.com/szlcsc/1809140220_UNI-ROYAL-Uniroyal-Elec-0603WAJ0103T5E_C15401.pdf" H 3650 3300 50  0001 C CNN
-F 4 "https://datasheet.lcsc.com/szlcsc/1809140220_UNI-ROYAL-Uniroyal-Elec-0603WAJ0103T5E_C15401.pdf" H 3650 3300 50  0001 C CNN "Description"
+F 4 "10kΩ ±5% 0.1W ±100ppm/℃ 0603 Chip Resistor - Surface Mount RoHS" H 3650 3300 50  0001 C CNN "Description"
 F 5 "C15401" H 3650 3300 50  0001 C CNN "LCSC Part #"
 F 6 "UNI-ROYAL(Uniroyal Elec)" H 3650 3300 50  0001 C CNN "Manufacturer"
@@
 F 7 "-" H 3850 3800 50  0001 C CNN "Maximum Value"
 F 8 "-" H 3850 3800 50  0001 C CNN "Mfr.Part #"
-F 9 "-" H 3850 3800 50  0001 C CNN "Package Reference"
+F 9 "2.54mm 1x2" H 3850 3800 50  0001 C CNN "Package Reference"
 	1    3850 3800
 	1    0    0    -1
@@
 F 2 "Resistor_SMD:R_0603_1608Metric_Pad0.98x0.95mm_HandSolder" V 7730 3350 50  0001 C CNN
 F 3 "https://datasheet.lcsc.com/szlcsc/1809140220_UNI-ROYAL-Uniroyal-Elec-0603WAJ0103T5E_C15401.pdf" H 7800 3350 50  0001 C CNN
-F 4 "https://datasheet.lcsc.com/szlcsc/1809140220_UNI-ROYAL-Uniroyal-Elec-0603WAJ0103T5E_C15401.pdf" H 7800 3350 50  0001 C CNN "Description"
+F 4 "10kΩ ±5% 0.1W ±100ppm/℃ 0603 Chip Resistor - Surface Mount RoHS" H 7800 3350 50  0001 C CNN "Description"
 F 5 "C15401" H 7800 3350 50  0001 C CNN "LCSC Part #"
 F 6 "UNI-ROYAL(Uniroyal Elec)" H 7800 3350 50  0001 C CNN "Manufacturer"
@@
 F 7 "-" H 8000 3850 50  0001 C CNN "Maximum Value"
 F 8 "-" H 8000 3850 50  0001 C CNN "Mfr.Part #"
-F 9 "-" H 8000 3850 50  0001 C CNN "Package Reference"
+F 9 "2.54mm 1x2" H 8000 3850 50  0001 C CNN "Package Reference"
 	1    8000 3850
 	1    0    0    -1

Commit message: PCB completed (added silkscreen more)
Parts:
- J501: value Conn_01x02_Female -> S1/U
- J502: value Conn_01x02_Female -> S2/D
Changed lines of the file:
@@
 P 3850 3800
 F 0 "J501" H 3900 3900 50  0000 L CNN
-F 1 "Conn_01x02_Female" H 3900 3800 50  0000 L CNN
+F 1 "S1/U" H 3900 3800 50  0000 L CNN
 F 2 "Connector_JST:JST_XH_B2B-XH-A_1x02_P2.50mm_Vertical" H 3850 3800 50  0001 C CNN
 F 3 "-" H 3850 3800 50  0001 C CNN
@@
 P 8000 3850
 F 0 "J502" H 8050 3950 50  0000 L CNN
-F 1 "Conn_01x02_Female" H 8050 3850 50  0000 L CNN
+F 1 "S2/D" H 8050 3850 50  0000 L CNN
 F 2 "Connector_JST:JST_XH_B2B-XH-A_1x02_P2.50mm_Vertical" H 8000 3850 50  0001 C CNN
 F 3 "-" H 8000 3850 50  0001 C CNN

Commit message: Rev 2 completed, todo check all and remove not needed filed
Parts:
- J401: renamed from J501; Description - -> (none); LCSC Part # - -> (none); Manufacturer - -> (none); Maximum Value - -> (none); Mfr.Part # - -> (none)
- J402: renamed from J502; Description - -> (none); LCSC Part # - -> (none); Manufacturer - -> (none); Maximum Value - -> (none); Mfr.Part # - -> (none)
- R401: renamed from R501; Description 10kΩ ±5% 0.1W ±100ppm/℃ 0603 Chip Resistor - Surface Mount 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 -> (none); LCSC (none) -> C25804; LCSC Part # C15401 -> (none); Manufacturer UNI-ROYAL(Uniroyal Elec) -> (none); Mfr.Part # 0603WAJ0103T5E -> (none)
- R402: renamed from R502; Description 10kΩ ±5% 0.1W ±100ppm/℃ 0603 Chip Resistor - Surface Mount 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 -> (none); LCSC (none) -> C25804; LCSC Part # C15401 -> (none); Manufacturer UNI-ROYAL(Uniroyal Elec) -> (none); Mfr.Part # 0603WAJ0103T5E -> (none)
Changed lines of the file:
@@
 $Descr A4 11693 8268
 encoding utf-8
-Sheet 5 8
+Sheet 4 8
 Title "Electra Project"
-Date "2021-03-21"
-Rev "1"
+Date "2021-04-01"
+Rev "2.0"
 Comp "Grehasopt"
 Comment1 "https://github.com/Grehasopt/Electra"
@@
 out2
 $Comp
-L Device:R R501
-U 1 1 609727A9
-P 3650 3300
-F 0 "R501" H 3720 3346 50  0000 L CNN
-F 1 "10K" V 3650 3200 50  0000 L CNN
-F 2 "Resistor_SMD:R_0603_1608Metric_Pad0.98x0.95mm_HandSolder" V 3580 3300 50  0001 C CNN
-F 3 "https://datasheet.lcsc.com/szlcsc/1809140220_UNI-ROYAL-Uniroyal-Elec-0603WAJ0103T5E_C15401.pdf" H 3650 3300 50  0001 C CNN
-F 4 "10kΩ ±5% 0.1W ±100ppm/℃ 0603 Chip Resistor - Surface Mount RoHS" H 3650 3300 50  0001 C CNN "Description"
-F 5 "C15401" H 3650 3300 50  0001 C CNN "LCSC Part #"
-F 6 "UNI-ROYAL(Uniroyal Elec)" H 3650 3300 50  0001 C CNN "Manufacturer"
-F 7 "0.1W" H 3650 3300 50  0001 C CNN "Maximum Value"
-F 8 "0603WAJ0103T5E" H 3650 3300 50  0001 C CNN "Mfr.Part #"
-F 9 "0603" H 3650 3300 50  0001 C CNN "Package Reference"
-	1    3650 3300
-	1    0    0    -1
-$EndComp
-$Comp
-L power:GND #PWR0502
+L power:GND #PWR0402
 U 1 1 60973678
 P 3650 4400
-F 0 "#PWR0502" H 3650 4150 50  0001 C CNN
+F 0 "#PWR0402" H 3650 4150 50  0001 C CNN
 F 1 "GND" H 3655 4227 50  0000 C CNN
 F 2 "" H 3650 4400 50  0001 C CNN
@@
 $EndComp
 $Comp
-L Connector:Conn_01x02_Female J501
+L Connector:Conn_01x02_Female J401
 U 1 1 6097414A
 P 3850 3800
-F 0 "J501" H 3900 3900 50  0000 L CNN
+F 0 "J401" H 3900 3900 50  0000 L CNN
 F 1 "S1/U" H 3900 3800 50  0000 L CNN
 F 2 "Connector_JST:JST_XH_B2B-XH-A_1x02_P2.50mm_Vertical" H 3850 3800 50  0001 C CNN
-F 3 "-" H 3850 3800 50  0001 C CNN
-F 4 "-" H 3850 3800 50  0001 C CNN "Description"
-F 5 "-" H 3850 3800 50  0001 C CNN "LCSC Part #"
-F 6 "-" H 3850 3800 50  0001 C CNN "Manufacturer"
-F 7 "-" H 3850 3800 50  0001 C CNN "Maximum Value"
-F 8 "-" H 3850 3800 50  0001 C CNN "Mfr.Part #"
-F 9 "2.54mm 1x2" H 3850 3800 50  0001 C CNN "Package Reference"
+F 3 "~" H 3850 3800 50  0001 C CNN
+F 4 "2.54mm 1x2" H 3850 3800 50  0001 C CNN "Package Reference"
 	1    3850 3800
 	1    0    0    -1
@@
 	3650 3600 3650 3800
 $Comp
-L Device:R R502
+L Device:R R402
 U 1 1 6097B75B
 P 7800 3350
-F 0 "R502" H 7870 3396 50  0000 L CNN
+F 0 "R402" H 7870 3396 50  0000 L CNN
 F 1 "10K" V 7800 3250 50  0000 L CNN
 F 2 "Resistor_SMD:R_0603_1608Metric_Pad0.98x0.95mm_HandSolder" V 7730 3350 50  0001 C CNN
-F 3 "https://datasheet.lcsc.com/szlcsc/1809140220_UNI-ROYAL-Uniroyal-Elec-0603WAJ0103T5E_C15401.pdf" H 7800 3350 50  0001 C CNN
-F 4 "10kΩ ±5% 0.1W ±100ppm/℃ 0603 Chip Resistor - Surface Mount RoHS" H 7800 3350 50  0001 C CNN "Description"
-F 5 "C15401" H 7800 3350 50  0001 C CNN "LCSC Part #"
-F 6 "UNI-ROYAL(Uniroyal Elec)" H 7800 3350 50  0001 C CNN "Manufacturer"
-F 7 "0.1W" H 7800 3350 50  0001 C CNN "Maximum Value"
-F 8 "0603WAJ0103T5E" H 7800 3350 50  0001 C CNN "Mfr.Part #"
-F 9 "0603" H 7800 3350 50  0001 C CNN "Package Reference"
+F 3 "~" H 7800 3350 50  0001 C CNN
+F 4 "C25804" H 7800 3350 50  0001 C CNN "LCSC"
+F 5 "0.1W" H 7800 3350 50  0001 C CNN "Maximum Value"
+F 6 "0603" H 7800 3350 50  0001 C CNN "Package Reference"
 	1    7800 3350
 	1    0    0    -1
 $EndComp
 $Comp
-L power:GND #PWR0504
+L power:GND #PWR0404
 U 1 1 6097B767
 P 7800 4450
-F 0 "#PWR0504" H 7800 4200 50  0001 C CNN
+F 0 "#PWR0404" H 7800 4200 50  0001 C CNN
 F 1 "GND" H 7805 4277 50  0000 C CNN
 F 2 "" H 7800 4450 50  0001 C CNN
@@
 $EndComp
 $Comp
-L Connector:Conn_01x02_Female J502
+L Connector:Conn_01x02_Female J402
 U 1 1 6097B76D
 P 8000 3850
-F 0 "J502" H 8050 3950 50  0000 L CNN
+F 0 "J402" H 8050 3950 50  0000 L CNN
 F 1 "S2/D" H 8050 3850 50  0000 L CNN
 F 2 "Connector_JST:JST_XH_B2B-XH-A_1x02_P2.50mm_Vertical" H 8000 3850 50  0001 C CNN
-F 3 "-" H 8000 3850 50  0001 C CNN
-F 4 "-" H 8000 3850 50  0001 C CNN "Description"
-F 5 "-" H 8000 3850 50  0001 C CNN "LCSC Part #"
-F 6 "-" H 8000 3850 50  0001 C CNN "Manufacturer"
-F 7 "-" H 8000 3850 50  0001 C CNN "Maximum Value"
-F 8 "-" H 8000 3850 50  0001 C CNN "Mfr.Part #"
-F 9 "2.54mm 1x2" H 8000 3850 50  0001 C CNN "Package Reference"
+F 3 "~" H 8000 3850 50  0001 C CNN
+F 4 "2.54mm 1x2" H 8000 3850 50  0001 C CNN "Package Reference"
 	1    8000 3850
 	1    0    0    -1
@@
 Reed Switch 2
 $Comp
-L power:VCC #PWR0501
+L power:VCC #PWR0401
 U 1 1 60982198
 P 3650 2900
-F 0 "#PWR0501" H 3650 2750 50  0001 C CNN
+F 0 "#PWR0401" H 3650 2750 50  0001 C CNN
 F 1 "VCC" H 3665 3073 50  0000 C CNN
 F 2 "" H 3650 2900 50  0001 C CNN
@@
 $EndComp
 $Comp
-L power:VCC #PWR0503
+L power:VCC #PWR0403
 U 1 1 60982984
 P 7800 2950
-F 0 "#PWR0503" H 7800 2800 50  0001 C CNN
+F 0 "#PWR0403" H 7800 2800 50  0001 C CNN
 F 1 "VCC" H 7815 3123 50  0000 C CNN
 F 2 "" H 7800 2950 50  0001 C CNN
@@
 	1    0    0    -1
 $EndComp
+$Comp
+L Device:R R401
+U 1 1 609727A9
+P 3650 3300
+F 0 "R401" H 3720 3346 50  0000 L CNN
+F 1 "10K" V 3650 3200 50  0000 L CNN
+F 2 "Resistor_SMD:R_0603_1608Metric_Pad0.98x0.95mm_HandSolder" V 3580 3300 50  0001 C CNN
+F 3 "~" H 3650 3300 50  0001 C CNN
+F 4 "C25804" H 3650 3300 50  0001 C CNN "LCSC"
+F 5 "0.1W" H 3650 3300 50  0001 C CNN "Maximum Value"
+F 6 "0603" H 3650 3300 50  0001 C CNN "Package Reference"
+	1    3650 3300
+	1    0    0    -1
+$EndComp
