File: pcb/Electra/Relay2.sch (KiCad schematic (older format))
At the start: 9 parts, among them J301 Screw_Terminal_01x03, K301 RAYEX-L90, Q301 Q_NPN_EBC

Commit message: PCB Ver 1 completed (TODO: Check)
Parts:
- removed K301: RAYEX-L90, Relay_THT:Relay_SPDT_Finder_36.11, symbol Relay:RAYEX-L90
- added K301: FINDER-36.11, Relay_THT:Relay_SPDT_Finder_36.11, symbol Relay:FINDER-36.11
- D302: footprint (none) -> Diode_SMD:D_SOD-323; Description (none) -> 85V 200mA 1.25V @ 150mA SOD-323 Diodes - General Purpose Ro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; LCSC Part # (none) -> C89953; Manufacturer (none) -> Nexperia; Maximum Value (none) -> 200mA; Mfr.Part # (none) -> BAS416,115; Package Reference (none) -> SOD-323
Connections:
- net +5V: now also K301.A1
- net Relay-Common: now also K301.11
- net Relay-Normal-Close: now also K301.12
- net Relay-Normal-Open: now also K301.14
- net at D302.1 (K), JP301.2, Q301.3 (C): now also K301.A2
Changed lines of the file:
@@
 $Descr A4 11693 8268
 encoding utf-8
-Sheet 3 7
+Sheet 3 8
 Title "Electra Project"
 Date "2021-03-21"
@@
 Comment4 ""
 $EndDescr
-$Comp
-L Relay:RAYEX-L90 K?
-U 1 1 607D3AA5
-P 6050 3550
-AR Path="/607D3AA5" Ref="K?"  Part="1"
-AR Path="/6072D929/607D3AA5" Ref="K?"  Part="1"
-AR Path="/60BEC19B/607D3AA5" Ref="K?"  Part="1"
-AR Path="/6079F8F1/607D3AA5" Ref="K301"  Part="1"
-F 0 "K301" H 6600 3650 50  0000 C CNN
-F 1 "RAYEX-L90" H 6700 3550 50  0000 C CNN
-F 2 "Relay_THT:Relay_SPDT_Finder_36.11" H 6500 3500 50  0001 L CNN
-F 3 "https://datasheet.lcsc.com/szlcsc/1912111437_HF-Xiamen-Hongfa-Electroacoustic-HF3FF-005-1ZS_C399562.pdf" H 6400 4550 50  0001 L CNN
-F 4 "General Purpose Non Latching 5VDC SPDT Through Hole Relays RoHS" H 6050 3550 50  0001 C CNN "Description"
-F 5 "C399562" H 6050 3550 50  0001 C CNN "LCSC Part #"
-F 6 " HF(Xiamen Hongfa Electroacoustic)" H 6050 3550 50  0001 C CNN "Manufacturer"
-F 7 "10A" H 6050 3550 50  0001 C CNN "Maximum Value"
-F 8 "HF3FF/005-1ZS" H 6050 3550 50  0001 C CNN "Mfr.Part #"
-F 9 "-" H 6050 3550 50  0001 C CNN "Package Reference"
-	1    6050 3550
-	1    0    0    -1
-$EndComp
 Text Label 6450 2900 0    50   ~ 10
 Relay-Normal-Close
@@
 F 0 "D302" V 5450 3900 50  0000 R CNN
 F 1 "DIODE" V 5350 3900 50  0000 R CNN
-F 2 "" H 5400 3550 50  0001 C CNN
-F 3 "~" H 5400 3550 50  0001 C CNN
+F 2 "Diode_SMD:D_SOD-323" H 5400 3550 50  0001 C CNN
+F 3 "https://datasheet.lcsc.com/szlcsc/1912111437_Nexperia-BAS416-115_C89953.pdf" H 5400 3550 50  0001 C CNN
+F 4 "85V 200mA 1.25V @ 150mA SOD-323 Diodes - General Purpose RoHS" H 5400 3550 50  0001 C CNN "Description"
+F 5 "C89953" H 5400 3550 50  0001 C CNN "LCSC Part #"
+F 6 "Nexperia" H 5400 3550 50  0001 C CNN "Manufacturer"
+F 7 "200mA" H 5400 3550 50  0001 C CNN "Maximum Value"
+F 8 "BAS416,115" H 5400 3550 50  0001 C CNN "Mfr.Part #"
+F 9 "SOD-323" H 5400 3550 50  0001 C CNN "Package Reference"
 	1    5400 3550
 	0    -1   -1   0
@@
 	6350 3150 6450 3150
 Wire Wire Line
-	6150 3150 6150 2900
-Wire Wire Line
 	6150 2900 6450 2900
 $Comp
@@
 	0    1    1    0
 $EndComp
+$Comp
+L Relay:FINDER-36.11 K301
+U 1 1 606462B6
+P 6050 3550
+F 0 "K301" H 6480 3596 50  0000 L CNN
+F 1 "FINDER-36.11" H 6480 3505 50  0000 L CNN
+F 2 "Relay_THT:Relay_SPDT_Finder_36.11" H 7320 3520 50  0001 C CNN
+F 3 "https://datasheet.lcsc.com/szlcsc/1912111437_HF-Xiamen-Hongfa-Electroacoustic-HF3FF-005-1ZS_C399562.pdf" H 6050 3550 50  0001 C CNN
+F 4 "General Purpose Non Latching 5VDC SPDT Through Hole Relays RoHS" H 6050 3550 50  0001 C CNN "Description"
+F 5 "C399562" H 6050 3550 50  0001 C CNN "LCSC Part #"
+F 6 " HF(Xiamen Hongfa Electroacoustic)" H 6050 3550 50  0001 C CNN "Manufacturer"
+F 7 "10A" H 6050 3550 50  0001 C CNN "Maximum Value"
+F 8 "HF3FF/005-1ZS" H 6050 3550 50  0001 C CNN "Mfr.Part #"
+F 9 "Finder_36.11" H 6050 3550 50  0001 C CNN "Package Reference"
+	1    6050 3550
+	1    0    0    -1
+$EndComp
+Wire Wire Line
+	5850 3950 5850 3850
+Wire Wire Line
+	6250 3950 6250 3850
+Wire Wire Line
+	5850 3250 5850 3150
+Wire Wire Line
+	6150 2900 6150 3250
+Wire Wire Line
+	6350 3250 6350 3150
 $EndSCHEMATC

Commit message: PCB completed (added silkscreen more)
Parts:
- D301: value LED -> R2; Description Red 615~630nm 0603 Light Emitting Diodes (LED) RoHS -> LIGHT EMITTING DIODES (LED) RED 520~625NM 90~100MCD@20MA TO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; LCSC Part # C84263 -> C2286; Manufacturer Foshan NationStar Optoelectronics -> Hubei KENTO Elec
- D302: value DIODE -> 200mA
- J301: value Screw_Terminal_01x03 -> Relay 2/D
- TP301: value Test Relay -> T2
Changed lines of the file:
@@
 AR Path="/6079F8F1/60C4940A" Ref="D302"  Part="1"
 F 0 "D302" V 5450 3900 50  0000 R CNN
-F 1 "DIODE" V 5350 3900 50  0000 R CNN
+F 1 "200mA" V 5350 3900 50  0000 R CNN
 F 2 "Diode_SMD:D_SOD-323" H 5400 3550 50  0001 C CNN
 F 3 "https://datasheet.lcsc.com/szlcsc/1912111437_Nexperia-BAS416-115_C89953.pdf" H 5400 3550 50  0001 C CNN
@@
 P 9300 3700
 F 0 "J301" H 9380 3742 50  0000 L CNN
-F 1 "Screw_Terminal_01x03" H 9380 3651 50  0000 L CNN
+F 1 "Relay 2/D" H 9380 3651 50  0000 L CNN
 F 2 "TerminalBlock:TerminalBlock_bornier-3_P5.08mm" H 9300 3700 50  0001 C CNN
 F 3 "~" H 9300 3700 50  0001 C CNN
@@
 U 1 1 60C4940E
 P 3200 4550
-F 0 "TP301" H 3050 4900 50  0000 L CNN
-F 1 "Test Relay" H 3050 4800 50  0000 L CNN
+F 0 "TP301" H 3150 4900 50  0000 L CNN
+F 1 "T2" H 3150 4800 50  0000 L CNN
 F 2 "TestPoint:TestPoint_Pad_D1.5mm" H 3400 4550 50  0001 C CNN
 F 3 "-" H 3400 4550 50  0001 C CNN
@@
 P 4300 3200
 F 0 "D301" V 4339 3082 50  0000 R CNN
-F 1 "LED" V 4248 3082 50  0000 R CNN
+F 1 "R2" V 4248 3082 50  0000 R CNN
 F 2 "LED_SMD:LED_0603_1608Metric_Pad1.05x0.95mm_HandSolder" H 4300 3200 50  0001 C CNN
-F 3 "https://datasheet.lcsc.com/szlcsc/2008201032_Foshan-NationStar-Optoelectronics-NCD0603R1_C84263.pdf" H 4300 3200 50  0001 C CNN
-F 4 "Red 615~630nm 0603 Light Emitting Diodes (LED) RoHS" H 4300 3200 50  0001 C CNN "Description"
-F 5 "C84263" H 4300 3200 50  0001 C CNN "LCSC Part #"
-F 6 "Foshan NationStar Optoelectronics" H 4300 3200 50  0001 C CNN "Manufacturer"
+F 3 "https://datasheet.lcsc.com/szlcsc/Hubei-KENTO-Elec-KT-0603R_C2286.pdf" H 4300 3200 50  0001 C CNN
+F 4 "LIGHT EMITTING DIODES (LED) RED 520~625NM 90~100MCD@20MA TOP VIEW 0603 ROHS" H 4300 3200 50  0001 C CNN "Description"
+F 5 "C2286" H 4300 3200 50  0001 C CNN "LCSC Part #"
+F 6 "Hubei KENTO Elec" H 4300 3200 50  0001 C CNN "Manufacturer"
 F 7 "25mA" H 4300 3200 50  0001 C CNN "Maximum Value"
 F 8 "NCD0603R1" H 4300 3200 50  0001 C CNN "Mfr.Part #"

Commit message: Rev 2 completed, todo check all and remove not needed filed
Parts:
- D301: Description LIGHT EMITTING DIODES (LED) RED 520~625NM 90~100MCD@20MA TO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 -> RED; LCSC (none) -> C2286; LCSC Part # C2286 -> (none); Manufacturer Hubei KENTO Elec -> (none); Maximum Value 25mA -> 19mA; Mfr.Part # NCD0603R1 -> (none)
- D302: footprint Diode_SMD:D_SOD-323 -> Diode_SMD:D_MiniMELF; Description 85V 200mA 1.25V @ 150mA SOD-323 Diodes - General Purpose Ro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 -> (none); LCSC (none) -> C9808; LCSC Part # C89953 -> (none); Manufacturer Nexperia -> (none); Mfr.Part # BAS416,115 -> (none); Package Reference SOD-323 -> LL-34
- J301: LCSC (none) -> C8425; Package Reference (none) -> 5.08mm
- JP301: Description - -> (none); LCSC Part # - -> (none); Manufacturer - -> (none); Maximum Value - -> (none); Mfr.Part # - -> (none)
- K301: LCSC (none) -> C399562; LCSC Part # C399562 -> (none); Manufacturer HF(Xiamen Hongfa Electroacoustic) -> (none); Mfr.Part # HF3FF/005-1ZS -> (none)
- Q301: LCSC (none) -> C75568; LCSC Part # C75568 -> (none); Manufacturer Nexperia -> (none); Maximum Value 100mA -> 100mA; Mfr.Part # BC847W,115 -> (none)
- R301: Description 1kΩ ±1% 0.1W ±100ppm/℃ 0603 Chip Resistor - Surface Mount R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 -> (none); LCSC (none) -> C21190; LCSC Part # C21190 -> (none); Manufacturer UNI-ROYAL(Uniroyal Elec) -> (none); Mfr.Part # 0603WAF1001T5E -> (none)
- R302: value 150 -> 68; Description 150Ω ±1% 0.1W ±100ppm/℃ 0603 Chip Resistor - Surface Mount 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 -> (none); LCSC (none) -> C27592; LCSC Part # C103302 -> (none); Manufacturer RALEC -> (none); Mfr.Part # RTT031500FTP -> (none)
- TP301: LCSC Part # - -> (none); Manufacturer - -> (none); Mfr.Part # - -> (none)

Commit message: Minor fixes on schematic and pcb fix bjt netlist + ac main voltage to both sides (Rev 2.1)
Parts:
- Q301: symbol Device:Q_NPN_EBC -> Device:Q_NPN_BEC
Connections:
- net GND: now also Q301.2 (E); no longer Q301.1 (E)
- net at R301.1: now also Q301.1 (B); no longer Q301.2 (B)
Changed lines of the file:
@@
 Sheet 3 8
 Title "Electra Project"
-Date "2021-04-01"
-Rev "2.0"
+Date "2021-05-04"
+Rev "2.1"
 Comp "Grehasopt"
 Comment1 "https://github.com/Grehasopt/Electra"
@@
 $EndComp
 $Comp
-L Device:Q_NPN_EBC Q?
+L Device:Q_NPN_BEC Q?
 U 1 1 60678E78
 P 4200 4650
